Commit message: 20250706updates

File: description/inertial_macros.xacro (robot description, xacro)
@@ -1,31 +1,33 @@
 <?xml version="1.0"?>
-<robot xmlns:xacro="http://www.ros.org/wiki/xacro" >
-    <!-- Specify some standard inertial calculations https://en.wikipedia.org/wiki/List_of_moments_of_inertia -->
+<robot xmlns:xacro="http://www.ros.org/wiki/xacro">
+    <!-- filename: inertial_macros.xacro -->
+    <!-- Specify some standard inertial calculations
+    https://en.wikipedia.org/wiki/List_of_moments_of_inertia -->
     <!-- These make use of xacro's mathematical functionality -->
     <xacro:macro name="inertial_sphere" params="mass radius *origin">
         <inertial>
-            <xacro:insert_block name="origin"/>
+            <xacro:insert_block name="origin" />
             <mass value="${mass}" />
             <inertia ixx="${(2/5) * mass * (radius*radius)}" ixy="0.0" ixz="0.0"
-                    iyy="${(2/5) * mass * (radius*radius)}" iyz="0.0"
-                    izz="${(2/5) * mass * (radius*radius)}" />
+                iyy="${(2/5) * mass * (radius*radius)}" iyz="0.0"
+                izz="${(2/5) * mass * (radius*radius)}" />
         </inertial>
     </xacro:macro>
     <xacro:macro name="inertial_box" params="mass x y z *origin">
         <inertial>
-            <xacro:insert_block name="origin"/>
+            <xacro:insert_block name="origin" />
             <mass value="${mass}" />
             <inertia ixx="${(1/12) * mass * (y*y+z*z)}" ixy="0.0" ixz="0.0"
-                    iyy="${(1/12) * mass * (x*x+z*z)}" iyz="0.0"
-                    izz="${(1/12) * mass * (x*x+y*y)}" />
+                iyy="${(1/12) * mass * (x*x+z*z)}" iyz="0.0"
+                izz="${(1/12) * mass * (x*x+y*y)}" />
         </inertial>
     </xacro:macro>
     <xacro:macro name="inertial_cylinder" params="mass length radius *origin">
         <inertial>
-            <xacro:insert_block name="origin"/>
+            <xacro:insert_block name="origin" />
             <mass value="${mass}" />
             <inertia ixx="${(1/12) * mass * (3*radius*radius + length*length)}" ixy="0.0" ixz="0.0"
-                    iyy="${(1/12) * mass * (3*radius*radius + length*length)}" iyz="0.0"
-                    izz="${(1/2) * mass * (radius*radius)}" />
+                iyy="${(1/12) * mass * (3*radius*radius + length*length)}" iyz="0.0"
+                izz="${(1/2) * mass * (radius*radius)}" />
         </inertial>
     </xacro:macro>

File: description/robot.urdf.xacro (robot description, xacro)
@@ -1,5 +1,8 @@
 <?xml version="1.0"?>
-<robot xmlns:xacro="http://www.ros.org/wiki/xacro"  name="robot">
-    <xacro:include filename="robot_core.xacro"/>
-    <xacro:include filename="inertial_macros.xacro"/>
+<robot xmlns:xacro="http://www.ros.org/wiki/xacro" name="robot">
+    <!-- filename: robot.urdf.xacro -->
+    <xacro:include filename="robot_core.xacro" />
+    <xacro:include filename="inertial_macros.xacro" />
+    <xacro:include filename="gazebo_control.xacro" />
+    <topic>/model/labrobot/cmd_vel</topic>
 </robot>

File: description/robot_core.xacro (robot description, xacro)
@@ -42,11 +42,14 @@
     <!-- if tires are touching ground, then base is offset by 52.5mm    -->
     <xacro:property name="chassis_z"
-        value="${(chassis_height / 2) + motor_mount_offset - wheel_radius}" />
+        value="${(chassis_height / 2) + motor_mount_offset - wheel_radius}"
+        />
     <!--
         origin should be center of the wheelbase axis, wheel radius from the front of the chassis
     -->
-    <xacro:property name="wheelbase_x" value="${(chassis_depth / 2) - wheel_radius}" />
-    <xacro:property name="wheelbase_y" value="${(chassis_width / 2) + (wheel_length/2)}" />
-    <!-- BASE LINK -->
+    <xacro:property name="wheelbase_x" value="${chassis_depth / 2}" />
+    <xacro:property name="wheelbase_y" value="${chassis_width / 2}" />
+    <xacro:property name="wheel_y" value="${wheelbase_y + (wheel_length / 2)}" />
+    <xacro:property name="caster_x" value="- ${chassis_width / 3} - ${wheel_radius}" />
+   <!-- BASE LINK -->
     <link name="base_link">
     </link>
@@ -76,14 +79,17 @@
         </xacro:inertial_box>
     </link>
+    <gazebo reference="chassis">
+        <material>Gazebo/Orange</material>
+    </gazebo>
     <!-- LEFT WHEEL Joint + Link -->
-    <joint name="left wheel_to_base_link" type="continuous">
+    <joint name="left_wheel_to_base_link" type="continuous">
         <parent link="base_link" />
         <child link="left_wheel" />
-        <origin xyz="${wheelbase_x} ${wheelbase_y} ${chassis_z}" rpy="0 0 0" />
-        <axis xyz="0 0 1" />
+        <origin xyz="-${wheel_radius} ${wheel_y} ${wheel_radius}" rpy="0 0 0" />
+        <axis xyz="0 1 0" />
     </joint>
     <link name="left_wheel">
         <visual>
-            <origin xyz="0 ${wheelbase_y} ${wheel_radius}" rpy="${pi/2} 0 0" />
+            <origin xyz="0 0 0" rpy="${pi/2} 0 0" />
             <geometry>
                 <cylinder radius="${wheel_radius}" length="${wheel_length}" />
@@ -92,5 +98,5 @@
         </visual>
         <collision>
-            <origin xyz="0 ${wheelbase_y} ${wheel_radius}" rpy="${pi/2} 0 0" />
+            <origin xyz="0 0 0" rpy="${pi/2} 0 0" />
             <geometry>
                 <cylinder radius="${wheel_radius}" length="${wheel_length}" />
@@ -98,18 +104,20 @@
         </collision>
         <xacro:inertial_cylinder mass="0.1" length="${wheel_length}" radius="${wheel_radius}">
-            <origin xyz="0 ${wheelbase_y} ${wheel_radius}" rpy="${pi/2} 0 0" />
+            <origin xyz="0 0 0" rpy="${pi/2} 0 0" />
         </xacro:inertial_cylinder>
     </link>
+    <gazebo reference="left_wheel">
+        <material>Gazebo/Blue</material>
+    </gazebo>
     <!-- RIGHT WHEEL Joint + Link -->
     <joint name="right_wheel_to_base_link" type="continuous">
         <parent link="base_link" />
         <child link="right_wheel" />
-        <!-- y is negative because of the left-handed coordinate system -->
-        <origin xyz="${wheelbase_x} -${wheelbase_y} ${chassis_z}" rpy="0 0 0" />
-        <axis xyz="0 0 1" />
+        <origin xyz="-${wheel_radius} -${wheel_y} ${wheel_radius}" rpy="0 0 0" />
+        <axis xyz="0 1 0" />
     </joint>
     <link name="right_wheel">
         <visual>
-            <origin xyz="0 -${wheelbase_y} ${wheel_radius}" rpy="${pi/2} 0 0" />
+            <origin xyz="0 0 0" rpy="${pi/2} 0 0" />
             <geometry>
                 <cylinder radius="${wheel_radius}" length="${wheel_length}" />
@@ -118,5 +126,5 @@
         </visual>
         <collision>
-            <origin xyz="0 -${wheelbase_y} ${wheel_radius}" rpy="${pi/2} 0 0" />
+            <origin xyz="0 0 0" rpy="${pi/2} 0 0" />
             <geometry>
                 <cylinder radius="${wheel_radius}" length="${wheel_length}" />
@@ -124,32 +132,36 @@
         </collision>
         <xacro:inertial_cylinder mass="0.1" length="${wheel_length}" radius="${wheel_radius}">
-            <origin xyz="0 -${wheelbase_y} ${wheel_radius}" rpy="${pi/2} 0 0" />
+            <origin xyz="0 0 0" rpy="${pi/2} 0 0" />
         </xacro:inertial_cylinder>
     </link>
-    <!-- CASTER WHEEL Joint + Link -->
-    <joint name="caster_wheel_to_base_link" type="continuous">
+    <gazebo reference="right_wheel">
+        <material>Gazebo/Blue</material>
+    </gazebo>
+    <!-- CASTER WHEEL (Spherical, for simulation stability) -->
+    <joint name="caster_wheel_joint" type="fixed">
         <parent link="base_link" />
         <child link="caster_wheel" />
-        <origin xyz="${wheelbase_x} 0 ${chassis_z}" rpy="0 0 0" />
-        <axis xyz="0 0 1" />
+        <origin xyz="-${(wheelbase_x * 2) - (wheel_radius)} 0 0.02" rpy="0 0 0" />
     </joint>
     <link name="caster_wheel">
         <visual>
-            <origin xyz="-${wheelbase_x * 2} 0 ${wheel_radius}" rpy="${pi/2} 0 0" />
             <geometry>
-                <cylinder radius="${wheel_radius}" length="${wheel_length}" />
+                <sphere radius="0.02" />
             </geometry>
-            <material name="blue" />
+            <material name="black" />
         </visual>
         <collision>
-            <origin xyz="-${wheelbase_x * 2} 0 ${wheel_radius}" rpy="${pi/2} 0 0" />
             <geometry>
-                <cylinder radius="${wheel_radius}" length="${wheel_length}" />
+                <sphere radius="0.02" />
             </geometry>
         </collision>
-        <xacro:inertial_cylinder mass="0.1" length="${wheel_length}" radius="${wheel_radius}">
-            <origin xyz="-${wheelbase_x * 2} 0 ${wheel_radius}" rpy="${pi/2} 0 0" />
-        </xacro:inertial_cylinder>
+        <xacro:inertial_sphere mass="0.1" radius="0.02">
+            <origin xyz="0 0 0" rpy="0 0 0" />
+        </xacro:inertial_sphere>
     </link>
-    <xacro:include filename="inertial_macros.xacro" />
+    <gazebo reference="caster_wheel">
+        <material>Gazebo/Blue</material>
+        <mu1 value="0.001" />
+        <mu2 value="0.001" />
+    </gazebo>
 </robot>
