Commit message: 7/26

File: description/lidar.xacro (robot description, xacro)
@@ -8,5 +8,5 @@
         <parent link="base_link" />
         <child link="lidar_frame" />
-        <origin xyz="-${lidar_sensor_diameter / 2} 0 ${chassis_height + lidar_sensor_height /2}" rpy="0 0 0" />
+        <origin xyz="${chassis_depth/2 - (lidar_sensor_diameter)} 0 ${chassis_height + 0.060}" rpy="0 0 0" />
     </joint>
     <link name="lidar_frame">

File: description/robot_core.xacro (robot description, xacro)
@@ -41,7 +41,5 @@
     <xacro:property name="motor_mount_offset" value="0.020" />
     <!-- if tires are touching ground, then base is offset by 52.5mm    -->
-    <xacro:property name="chassis_z"
-        value="${(chassis_height / 2) + motor_mount_offset - wheel_radius}"
-        />
+    <xacro:property name="chassis_z" value="${(wheel_radius + motor_mount_offset) + chassis_height / 2}" />
     <!--
         origin should be center of the wheelbase axis, wheel radius from the front of the chassis
@@ -58,9 +56,9 @@
         <parent link="base_link" />
         <child link="chassis" />
-        <origin xyz="0 0 ${wheel_radius}" rpy="0 0 0" />
+        <origin xyz="0 0 0" rpy="0 0 0" /> <!-- Centered on origin -->
     </joint>
     <link name="chassis">
         <visual>
-            <origin xyz="-${wheelbase_x} 0 ${chassis_z}" rpy="0 0 0" />
+            <origin xyz="0 0 ${chassis_z}" rpy="0 0 0" /> <!-- Centered on origin -->
             <geometry>
                 <box size="${chassis_depth} ${chassis_width} ${chassis_height}" />
@@ -69,5 +67,5 @@
         </visual>
         <collision>
-            <origin xyz="-${wheelbase_x} 0 ${chassis_z}" rpy="0 0 0" />
+            <origin xyz="0 0 ${chassis_z}" rpy="0 0 0" /> <!-- Centered on origin -->
             <geometry>
                 <box size="${chassis_depth} ${chassis_width} ${chassis_height}" />
@@ -76,5 +74,5 @@
         <xacro:inertial_box mass="7.5" x="${chassis_depth}" y="${chassis_width}"
             z="${chassis_height}">
-            <origin xyz="-${wheelbase_x} 0 ${chassis_z}" rpy="0 0 0" />
+            <origin xyz="0 0 ${chassis_z}" rpy="0 0 0" /> <!-- Centered on origin -->
         </xacro:inertial_box>
     </link>
@@ -86,5 +84,5 @@
         <parent link="base_link" />
         <child link="left_wheel" />
-        <origin xyz="-${wheel_radius} ${wheel_y} ${wheel_radius}" rpy="0 0 0" />
+        <origin xyz="0 ${wheel_y} ${wheel_radius}" rpy="0 0 0" />
         <axis xyz="0 1 0" />
     </joint>
@@ -114,5 +112,5 @@
         <parent link="base_link" />
         <child link="right_wheel" />
-        <origin xyz="-${wheel_radius} -${wheel_y} ${wheel_radius}" rpy="0 0 0" />
+        <origin xyz="0 -${wheel_y} ${wheel_radius}" rpy="0 0 0" />
         <axis xyz="0 1 0" />
     </joint>
@@ -139,10 +137,10 @@
     </gazebo>
     <!-- CASTER WHEEL (Spherical, for simulation stability) -->
-    <joint name="caster_wheel_joint" type="fixed">
+    <joint name="caster_wheel_f_joint" type="fixed">
         <parent link="base_link" />
-        <child link="caster_wheel" />
-        <origin xyz="-${(wheelbase_x * 2) - (wheel_radius)} 0 0.02" rpy="0 0 0" />
+        <child link="caster_wheel_f" />
+        <origin xyz="-${(wheelbase_x) - (wheel_radius)} 0 0.02" rpy="0 0 0" />
     </joint>
-    <link name="caster_wheel">
+    <link name="caster_wheel_f">
         <visual>
             <geometry>
@@ -160,5 +158,32 @@
         </xacro:inertial_sphere>
     </link>
-    <gazebo reference="caster_wheel">
+    <gazebo reference="caster_wheel_f">
+        <material>Gazebo/Blue</material>
+        <mu1 value="0.001" />
+        <mu2 value="0.001" />
+    </gazebo>
+    <!-- CASTER WHEEL (Spherical, for simulation stability) -->
+    <joint name="caster_wheel_b_joint" type="fixed">
+        <parent link="base_link" />
+        <child link="caster_wheel_b" />
+        <origin xyz="${(wheelbase_x) - (wheel_radius)} 0 0.02" rpy="0 0 0" />
+    </joint>
+    <link name="caster_wheel_b">
+        <visual>
+            <geometry>
+                <sphere radius="0.02" />
+            </geometry>
+            <material name="black" />
+        </visual>
+        <collision>
+            <geometry>
+                <sphere radius="0.02" />
+            </geometry>
+        </collision>
+        <xacro:inertial_sphere mass="0.1" radius="0.02">
+            <origin xyz="0 0 0" rpy="0 0 0" />
+        </xacro:inertial_sphere>
+    </link>
+    <gazebo reference="caster_wheel_b">
         <material>Gazebo/Blue</material>
         <mu1 value="0.001" />

Commit message: +lidar

File: description/lidar.xacro (robot description, xacro)
@@ -8,5 +8,5 @@
         <parent link="base_link" />
         <child link="lidar_frame" />
-        <origin xyz="${chassis_depth/2 - (lidar_sensor_diameter)} 0 ${chassis_height + 0.060}" rpy="0 0 0" />
+        <origin xyz="${chassis_depth/2 - (lidar_sensor_diameter)} 0 ${chassis_height + 0.060}" rpy="0 0 3.14" />
     </joint>
     <link name="lidar_frame">

File: description/robot_core.xacro (robot description, xacro)
@@ -190,3 +190,18 @@
         <mu2 value="0.001" />
     </gazebo>
+    <!-- FRONT MARKER (visual only) -->
+    <link name="front_marker">
+        <visual>
+            <origin xyz="${chassis_depth/2 + 0.05} 0 ${chassis_z + 0.05}" rpy="0 0 0" />
+            <geometry>
+                <cylinder radius="0.01" length="0.05" />
+            </geometry>
+            <material name="red" />
+        </visual>
+    </link>
+    <joint name="front_marker_joint" type="fixed">
+        <parent link="base_link" />
+        <child link="front_marker" />
+        <origin xyz="${chassis_depth/2 + 0.05} 0 ${chassis_z + 0.05}" rpy="0 0 0" />
+    </joint>
 </robot>

Commit message: +lidar

File: description/lidar.xacro (robot description, xacro)
@@ -12,5 +12,5 @@
     <link name="lidar_frame">
         <visual>
-            <origin xyz="0 0 0" rpy="0 0 0" />
+            <origin xyz="0 0 0" rpy="0 0 3.14" />
             <geometry>
                 <cylinder radius="${lidar_sensor_diameter / 2}" length="0.01" />
@@ -19,5 +19,5 @@
         </visual>
         <collision>
-            <origin xyz="0 0 0" rpy="0 0 0" />
+            <origin xyz="0 0 0" rpy="0 0 3.14" />
             <geometry>
                 <cylinder radius="${lidar_sensor_diameter / 2}" length="0.01" />

Commit message: +lidar

File: description/lidar.xacro (robot description, xacro)
@@ -8,9 +8,9 @@
         <parent link="base_link" />
         <child link="lidar_frame" />
-        <origin xyz="${chassis_depth/2 - (lidar_sensor_diameter)} 0 ${chassis_height + 0.060}" rpy="0 0 3.14" />
+        <origin xyz="${chassis_depth/2 - (lidar_sensor_diameter)} 0 ${chassis_height + 0.060}" rpy="0 0 0" />
     </joint>
     <link name="lidar_frame">
         <visual>
-            <origin xyz="0 0 0" rpy="0 0 3.14" />
+            <origin xyz="0 0 0" rpy="0 0 0" />
             <geometry>
                 <cylinder radius="${lidar_sensor_diameter / 2}" length="0.01" />
@@ -19,5 +19,5 @@
         </visual>
         <collision>
-            <origin xyz="0 0 0" rpy="0 0 3.14" />
+            <origin xyz="0 0 0" rpy="0 0 0" />
             <geometry>
                 <cylinder radius="${lidar_sensor_diameter / 2}" length="0.01" />

Commit message: +lidar

File: description/lidar.xacro (robot description, xacro)
@@ -8,5 +8,5 @@
         <parent link="base_link" />
         <child link="lidar_frame" />
-        <origin xyz="${chassis_depth/2 - (lidar_sensor_diameter)} 0 ${chassis_height + 0.060}" rpy="0 0 0" />
+        <origin xyz="${chassis_depth/2 - (lidar_sensor_diameter)} 0 ${chassis_height + 0.060}" rpy="0 0 3.14159" /> <!-- Rotated 180 degrees in yaw -->
     </joint>
     <link name="lidar_frame">
