Commit message: +camera, fixed picow main.py

File: description/camera.xacro (robot description, xacro)
@@ -1,9 +1,13 @@
 <?xml version="1.0"?>
 <robot xmlns:xacro="http://www.ros.org/wiki/xacro">
-  <!-- Place lidar just above chassis -->
+  <!-- Filename: camera.xacro -->
+  <!-- Define fallback properties - these will be overridden if already defined -->
+  <xacro:property name="chassis_depth" value="0.368" />
+  <xacro:property name="chassis_height" value="0.62" />
+  <!-- Place camera at front of chassis -->
   <joint name="camera_joint" type="fixed">
     <parent link="base_link" />
     <child link="camera_link" />
-    <origin xyz="${chassis_depth/2} 0 ${chassis_height + 0.060}" rpy="0 0 3.14159" />
+    <origin xyz="${chassis_depth/2 - 0.012} 0 ${chassis_height + 0.060}" rpy="0 0 0" />
   </joint>
   <link name="camera_link">
@@ -11,35 +15,46 @@
       <origin xyz="0 0 0" rpy="0 0 0" />
       <geometry>
-        <cylinder box="0.010 0.03 0.03" />
+        <box size="0.028 0.075 0.0175" /> <!-- 75mm x 28mm x 17.5mm -->
       </geometry>
       <material name="white" />
     </visual>
+    <collision>
+      <origin xyz="0 0 0" rpy="0 0 0" />
+      <geometry>
+        <box size="0.028 0.075 0.0175" />
+      </geometry>
+    </collision>
+    <inertial>
+      <origin xyz="0 0 0" rpy="0 0 0" />
+      <mass value="0.05" /> <!-- Approximate mass in kg -->
+      <inertia ixx="1e-5" ixy="0" ixz="0" iyy="1e-5" iyz="0" izz="1e-5" /> <!-- Simple inertia -->
+    </inertial>
   </link>
   <joint name="camera_optical_joint" type="fixed">
     <parent link="camera_link" />
     <child link="camera_link_optical" />
-    <origin xyz="0 0 0" rpy="${-pi/2} 0 ${pi/2}" />
+    <origin xyz="0 0 0" rpy="${-pi/2} 0 ${-pi/2}" />
   </joint>
   <link name="camera_link_optical" />
   <gazebo reference="camera_link">
     <material>Gazebo/White</material>
-    <!-- <sensor>
-      <name>camera</name>
-      <type>camera</type>
-      <update_rate>30</update_rate>
-      <topic>camera/image_raw</topic>
+    <sensor name="camera" type="camera">
+      <update_rate>10</update_rate>
       <always_on>1</always_on>
       <visualize>true</visualize>
+      <topic>camera/image_raw</topic>
       <camera>
-        <horizontal>
-          <resolution>640</resolution>
-          <fov>1.047</fov>
-        </horizontal>
-        <vertical>
-          <resolution>480</resolution>
-          <fov>0.785</fov>
-        </vertical>
+        <horizontal_fov>1.089</horizontal_fov>
+        <image>
+          <width>640</width>
+          <height>480</height>
+          <format>R8G8B8</format>
+        </image>
+        <clip>
+          <near>0.05</near>
+          <far>8.0</far>
+        </clip>
       </camera>
-    </sensor> -->
+    </sensor>
   </gazebo>
 </robot>

File: description/gazebo_control.xacro (robot description, xacro)
@@ -2,4 +2,7 @@
 <robot xmlns:xacro="http://www.ros.org/wiki/xacro">
     <!-- Gazebo DiffDrive plugin configuration for LabRobot -->
+    <!-- Define fallback properties - these will be overridden if already defined -->
+    <xacro:property name="wheelbase_y" value="0.1605" /> <!-- chassis_width/2 -->
+    <xacro:property name="wheel_radius" value="0.0325" /> <!-- wheel_diameter/2 -->
     <gazebo>
         <plugin name="gz::sim::systems::DiffDrive" filename="gz-sim-diff-drive-system">

File: description/lidar.xacro (robot description, xacro)
@@ -2,4 +2,7 @@
 <robot xmlns:xacro="http://www.ros.org/wiki/xacro">
     <!-- filename: lidar.xacro -->
+    <!-- Define fallback properties - these will be overridden if already defined -->
+    <xacro:property name="chassis_depth" value="0.368" />
+    <xacro:property name="chassis_height" value="0.62" />
     <xacro:property name="lidar_sensor_diameter" value="0.051" />
     <xacro:property name="lidar_sensor_height" value="0.045" />
@@ -8,5 +11,5 @@
         <parent link="base_link" />
         <child link="lidar_frame" />
-        <origin xyz="${chassis_depth/2 - (lidar_sensor_diameter)} 0 ${chassis_height + 0.060}" rpy="0 0 3.14159" /> <!-- Rotated 180 degrees in yaw -->
+        <origin xyz="${chassis_depth/2 - (lidar_sensor_diameter)} 0 ${chassis_height + 0.075}" rpy="0 0 3.14159" /> <!-- Rotated 180 degrees in yaw -->
     </joint>
     <link name="lidar_frame">
@@ -14,5 +17,5 @@
             <origin xyz="0 0 0" rpy="0 0 0" />
             <geometry>
-                <cylinder radius="${lidar_sensor_diameter / 2}" length="0.01" />
+                <cylinder radius="${lidar_sensor_diameter / 2}" length="0.05" />
             </geometry>
             <material name="white" />
