Commit message: fixed odom, joint_state_pub

File: description/gazebo_control.xacro (robot description, xacro)
@@ -15,7 +15,9 @@
             <odom_publish>true</odom_publish>
             <frame_id>odom</frame_id>
-            <child_frame_id>base_link</child_frame_id>
+            <child_frame_id>base_footprint</child_frame_id>
+            <tf_topic>/tf</tf_topic>
             <update_rate>50</update_rate>
             <publish_tf>true</publish_tf>
+            <publish_odom>true</publish_odom>
         </plugin>
     </gazebo>

File: description/robot.urdf.xacro (robot description, xacro)
@@ -6,9 +6,11 @@
     <xacro:include filename="gazebo_control.xacro" />
     <xacro:include filename="lidar.xacro" />
-    <xacro:include filename="camera.xacro" />
+    <!-- <xacro:include filename="camera.xacro" /> -->
+    <xacro:include filename="depth_camera.xacro" />
     <!-- Gazebo system plugins for sensors and joint state publisher -->
     <gazebo>
         <plugin name="gz::sim::systems::Sensors" filename="gz-sim-sensors-system" />
         <plugin name="gz::sim::systems::JointStatePublisher" filename="gz-sim-joint-state-publisher-system" />
+        <plugin name="gz::sim::systems::DiffDrive" filename="gz-sim-diff-drive-system" />
     </gazebo>
 </robot>

File: description/robot_core.xacro (robot description, xacro)
@@ -49,7 +49,16 @@
     <xacro:property name="wheel_y" value="${wheelbase_y + (wheel_length / 2)}" />
     <xacro:property name="caster_x" value="- ${chassis_width / 3} - ${wheel_radius}" />
-   <!-- BASE LINK -->
+   <!-- BASE FOOTPRINT - for odometry on ground plane -->
+    <link name="base_footprint">
+    </link>
+    <!-- BASE LINK -->
     <link name="base_link">
     </link>
+    <!-- Joint connecting base_footprint to base_link -->
+    <joint name="base_footprint_to_base_link" type="fixed">
+        <parent link="base_footprint" />
+        <child link="base_link" />
+        <origin xyz="0 0 ${wheel_radius}" rpy="0 0 0" />
+    </joint>
     <!-- CHASSIS  Joint + Link -->
     <joint name="chassis_to_base_link" type="fixed">
